Commit message: clean up of module | irreducible shooter fixes | urdf/launch files added

File: urdf/floor.urdf (robot description, URDF)
Before this commit: robot floor_description, 2 links, 1 joints
Links:
- link floor: geometry collision box size=4.0 6.0 0.1; visual box size=4.0 6.0 0.1

File: urdf/floor_obstacle.urdf (robot description, URDF)
Before this commit: robot floor_description, 3 links, 2 joints
Links:
- link floor: geometry collision box size=4.0 6.0 0.1; visual box size=4.0 6.0 0.1
